File: vakalan_gps_lorawan.kicad_pcb (KiCad board)
At the start: 2 copper layers, 147.5 x 90.1 mm, 64 parts, among them J1 Conn_01x08_Male, U1 BMM150, U2 TPS62A01DRLR_, U3 18650, U4 18650, U5 18650, U6 18650, U7 18650, U8 18650

Commit message: .
Parts:
- removed TP9: TestPoint_Probe, TestPoint:TestPoint_Pad_1.0x1.0mm
- added BZ1: Buzzer, Buzzer_Beeper:Buzzer_12x9.5RM7.6, F.Cu at (163.3, 134.4)
- added C12: 4.7uF, Capacitor_SMD:C_0805_2012Metric, F.Cu at (206.3, 139.5)
- added C13: 1uF, Capacitor_SMD:C_0805_2012Metric, F.Cu at (198.4, 145.1)
- added C14: 220Nf, Capacitor_SMD:C_0805_2012Metric, F.Cu at (142.9, 118.1)
- added C15: 0.1uF, Capacitor_SMD:C_0805_2012Metric, F.Cu at (142.9, 123.3)
- added D10: BAT54G, vakalan:BAT54G, F.Cu at (132.9, 119.6)
- added D7: D, vakalan:FM4006, F.Cu at (155.8, 146.1)
- added D8: D, vakalan:SS14, F.Cu at (198.4, 136.8)
- added D9: LED, LED_SMD:LED_0805_2012Metric, F.Cu at (112.9, 131.2)
- added L2: 10uH, vakalan:CDRH4D16-100M, F.Cu at (202.3, 133.0)
- added Q1: BUK9M11-40EX, Package_TO_SOT_SMD:LFPAK33, F.Cu at (146.9, 145.9)
- added R14: 10k, Resistor_SMD:R_0805_2012Metric, F.Cu at (204.2, 143.2)
- added R15: 0, Resistor_SMD:R_0805_2012Metric, F.Cu at (155.7, 141.6)
- added R16: 10k, Resistor_SMD:R_0805_2012Metric, F.Cu at (147.0, 142.2)
- added R17: 120k, Resistor_SMD:R_0805_2012Metric, F.Cu at (201.9, 143.2)
- added R18: 1M, Resistor_SMD:R_0805_2012Metric, F.Cu at (198.4, 142.9)
- added R19: 4.7k, Resistor_SMD:R_0805_2012Metric, F.Cu at (115.2, 131.2)
- added TP15: TestPoint_Probe, TestPoint:TestPoint_Pad_1.0x1.0mm, F.Cu at (143.6, 142.1)
- added TP16: TestPoint_Probe, TestPoint:TestPoint_Pad_1.0x1.0mm, F.Cu at (115.2, 127.5)
- added TP17: TestPoint_Probe, TestPoint:TestPoint_Pad_1.0x1.0mm, F.Cu at (54.7, 140.5)
- added TP18: TestPoint_Probe, TestPoint:TestPoint_Pad_1.0x1.0mm, F.Cu at (52.5, 140.5)
- added U9: AP3012, Package_TO_SOT_SMD:SOT-23-5, F.Cu at (202.4, 138.6)
- C4: value 0.1uF -> 10uF
- J1: footprint Connector_PinHeader_2.54mm:PinHeader_1x09_P2.54mm_Vertical -> Connector_PinHeader_2.54mm:PinHeader_1x09_P2.54mm_Vertical_SMD_Pin1Left
- JP1, JP2, JP3, JP4, JP5, JP6: footprint Connector_PinHeader_1.00mm:PinHeader_1x02_P1.00mm_Vertical -> Connector_PinHeader_2.54mm:PinHeader_1x02_P2.54mm_Vertical
- U1: value BMM150 -> IIS2MDCTR; footprint Package_CSP:WLCSP-12_1.56x1.56mm_P0.4mm -> vakalan:IIS2MDCTR
- moved R11 123.3 mm to (56.5, 115.0), turned to -90 degrees
- moved D5 112.3 mm to (178.2, 144.1), turned to -90 degrees
- moved JP5 100.7 mm to (178.4, 148.2)
- moved D2 100.2 mm to (178.6, 113.5), turned to 90 degrees
- moved TP8 98.5 mm to (196.2, 122.1), turned to 180 degrees
- moved JP2 97.6 mm to (178.8, 109.7), turned to 180 degrees
- moved TP7 97.4 mm to (191.7, 111.4)
- moved C8 95.1 mm to (57.4, 118.6)
- moved D1 73.2 mm to (22.7, 144.1), turned to -90 degrees
- moved TP4 72.7 mm to (53.9, 143.4)
- moved JP1 72.5 mm to (22.9, 148.0)
- moved U7 71.0 mm to (214.4, 139.4), turned to -90 degrees
- moved R8 65.7 mm to (190.8, 116.0)
- moved F1 65.2 mm to (215.9, 129.0), turned to 180 degrees
- moved TP14 65.1 mm to (141.3, 142.1), turned to -90 degrees
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Connections:
- J1 pad 3: RAK3172_UART2_TX -> RAK3172_RST
- J1 pad 4: RAK3172_UART2_RX -> RAK3172_BOOT0
- J1 pad 5: RAK3172_SWIO -> RAK3172_UART2_TX
- J1 pad 6: RAK3172_SWCLK -> RAK3172_UART2_RX
- J1 pad 7: RAK3172_BOOT0 -> RAK3172_SWIO
- J1 pad 8: RAK3172_RST -> RAK3172_SWCLK
- S2 pad 7: unconnected-(S2-Pad7) -> Net-(S2-Pad7)
- S2 pad 8: unconnected-(S2-Pad8) -> Net-(S2-Pad8)
- SOC1 pad 13: unconnected-(SOC1-Pad13) -> LED
- SOC1 pad 15: unconnected-(SOC1-Pad15) -> BUZZER
- SOC1 pad 19: unconnected-(SOC1-Pad19) -> AP3015_SHDN
- SOC1 pad 2: RAK3172_UART2_TX -> Net-(D10-Pad1)
- SOC1 pad 20: M10Q_EXINT -> M10Q_RESET_N
- SOC1 pad 25: BMM150_INT -> IIS2MDCTR_INT
- SOC1 pad 26: BMM150_DRDY -> unconnected-(SOC1-Pad26)
- SOC1 pad 30: M10Q_RESET_N -> M10Q_EXINT
- TP10 pad 1: BMM150_INT -> IIS2MDCTR_INT
- TP12 pad 1: M10Q_EXINT -> M10Q_RESET_N
- TP13 pad 1: M10Q_RESET_N -> M10Q_EXINT
Routing:
- net Net-(F1-Pad1): track 0.00 -> 544.5 mm
- net ADC_REF: track 0.00 -> 226.3 mm, vias 0 -> 4
- net SDA: track 0.00 -> 125.1 mm, vias 0 -> 5
- net SCL: track 0.00 -> 124.5 mm, vias 0 -> 3
- net AP3015_SHDN: track 0.00 -> 120.4 mm, vias 0 -> 2
- net M10Q_EXINT: track 0.00 -> 88.9 mm, vias 0 -> 2
- net M10Q_UART_RX: track 0.00 -> 84.0 mm
- net M10Q_RESET_N: track 0.00 -> 84.0 mm, vias 0 -> 2
- net M10Q_UART_TX: track 0.00 -> 82.1 mm
- net BATTERY: track 0.00 -> 74.2 mm, vias 0 -> 2
- net +3V0_MCU: track 0.00 -> 72.1 mm, vias 0 -> 2
- net BUZZER: track 0.00 -> 66.6 mm
- net Net-(C1-Pad1): track 0.00 -> 57.1 mm
- net +12V: track 0.00 -> 52.5 mm
- net +3V0_GPS: track 0.00 -> 31.7 mm
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- added copper zone on F.Cu, net +12V
- added copper zone on F.Cu, net ADC_REF
- added copper zone on B.Cu, net GND
- added copper zone on F.Cu, net GND
- added copper zone on F.Cu, net Net-(C1-Pad1)
- added copper zone on F.Cu, net Net-(D8-Pad1)
Other:
- board size 147.5 x 90.1 mm -> 248.3 x 59.6 mm
- board text added: "+"
- board text added: "-"
- board text added: "1"
- board text added: "3V0"
- board text added: "3V0_MCU"
- board text added: "9"
- board text added: "BATTERY(VOLT)"
- board text added: "BUZZER"
- board text added: "GND"
- board text added: "I2C_SCL"
- board text added: "I2C_SDA"
- board text added: "IIS2MDCTR_INT(MAG)"
- board text added: "J1"
- board text added: "LED"
- board text added: "LSM6D_INT1(ACCEL+GYR)"
- board text added: "LSM6D_INT2(ACCEL+GYR)"
- board text added: "M10Q_EXINT(GPS)"
- board text added: "M10Q_RESET_N(GPS)"
- board text added: "M10Q_SAFEBOOT(GPS)"
- board text added: "M10Q_TIMEPULSE(GPS)"
- board text added: "M10Q_UART_RX(GPS)"
- board text added: "M10Q_UART_TX(GPS)"
- board text added: "M3"
- board text added: "RAK3172_BOOT0"
- board text added: "RAK3172_RST"
- board text added: "RAK3172_SWCLK"
- board text added: "RAK3172_SWIO"
- board text added: "RAK3172_UART2_RX"
- board text added: "RAK3172_UART2_TX"
- board text added: "TP1"
- board text added: "TP10"
- board text added: "TP11"
- board text added: "TP12"
- board text added: "TP13"
- board text added: "TP14"
- board text added: "TP15"
- board text added: "TP16"
- board text added: "TP17"
- board text added: "TP18"
- board text added: "TP2"
- board text added: "TP3"
- board text added: "TP4"
- board text added: "TP5"
- board text added: "TP6"
- board text added: "TP7"
- board text added: "TP8"
